Commit message: siro_arm

File: src/siro_arm/urdf/arm1.urdf (robot description, URDF)
Before this commit: robot arm1, 3 links, 2 joints
Links:
- removed link base_link
- removed link link_1
- added link part1; collision mesh filename=package://siro_arm/models/meshes/collision/Ensamble_1.dae; visual mesh filename=package://siro_arm/models/meshes/visual/Ensamble_1.stl
- added link part2; collision mesh filename=package://siro_arm/models/meshes/collision/Ensamble_2.dae; visual mesh filename=package://siro_arm/models/meshes/visual/Ensamble_2.stl
- added link part3; collision mesh filename=package://siro_arm/models/meshes/collision/Ensamble_3.dae; visual mesh filename=package://siro_arm/models/meshes/visual/Ensamble_3.stl
- added link part4; collision mesh filename=package://siro_arm/models/meshes/collision/Ensamble_4.dae; visual mesh filename=package://siro_arm/models/meshes/visual/Ensamble_4.stl
- added link part5; collision mesh filename=package://siro_arm/models/meshes/collision/Ensamble_5.dae; visual mesh filename=package://siro_arm/models/meshes/visual/Ensamble_5.stl
- added link part6; collision mesh filename=package://siro_arm/models/meshes/collision/Ensamble_6.dae; visual mesh filename=package://siro_arm/models/meshes/visual/Ensamble_6.stl
Joints:
- removed joint fixed
- added joint fixed_joint: type fixed, parent world, child part1, origin xyz=0 0 0 rpy=0 0 0
- added joint joint_2: type revolute, parent part2, child part3, origin xyz=0.194649 0.152205 0.247295 rpy=0 0 0, axis 0 1 0, limit lower=-1.57 upper=1.57 effort=10 velocity=1.0
- added joint joint_3: type revolute, parent part3, child part4, origin xyz=0 0 1.23 rpy=0 0 0, axis 0 1 0, limit lower=-1.57 upper=1.57 effort=10 velocity=1.0
- added joint joint_4: type revolute, parent part4, child part5, origin xyz=1.2196 -0.401701 -0.009168 rpy=0 0 0, axis 0 1 0, limit lower=-1.57 upper=1.57 effort=10 velocity=1.0
- added joint joint_5: type revolute, parent part5, child part6, origin xyz=0.606218 0.228952 0.118208 rpy=0 -0.10853 0, axis 1 0 0, limit lower=-1.57 upper=1.57 effort=10 velocity=1.0
- joint joint_1: child link_1 -> part2; limit lower=-1.57 upper=1.57 effort=0 velocity=0.5 -> lower=-1.57 upper=1.57 effort=10 velocity=1.0; origin xyz=0 0 5 rpy=0 0 0 -> xyz=0 0 0.6367 rpy=0 0 0; parent base_link -> part1
