Commit message: siro_arm

File: src/siro_arm/urdf/siro_arm.urdf (robot description, URDF)
Before this commit: robot arm1, 7 links, 6 joints
Links:
- link part1: geometry collision mesh filename=package://siro_arm/meshes/collision/Ensamble_1.dae; visual mesh filename=package://siro_arm/meshes/visual/Ensamble_1.stl
- link part2: geometry collision mesh filename=package://siro_arm/meshes/collision/Ensamble_2.dae; visual mesh filename=package://siro_arm/meshes/visual/Ensamble_2.stl
- link part3: geometry collision mesh filename=package://siro_arm/meshes/collision/Ensamble_3.dae; visual mesh filename=package://siro_arm/meshes/visual/Ensamble_3.stl
- link part4: geometry collision mesh filename=package://siro_arm/meshes/collision/Ensamble_4.dae; visual mesh filename=package://siro_arm/meshes/visual/Ensamble_4.stl
- link part5: geometry collision mesh filename=package://siro_arm/meshes/collision/Ensamble_5.dae; visual mesh filename=package://siro_arm/meshes/visual/Ensamble_5.stl
- link part6: geometry collision mesh filename=package://siro_arm/meshes/collision/Ensamble_6.dae; visual mesh filename=package://siro_arm/meshes/visual/Ensamble_6.stl
